Commit message: Everything seems to be working correctly and the code is moving towards being cleaned up

File: assets/urdf/CubeBot.urdf (robot description, URDF)
Before this commit: robot CubeBot, 15 links, 14 joints
Links:
- added link WheelMarker_1, mass 0.01; visual box size=0.1 0.02 0.02
- added link WheelMarker_2, mass 0.01; visual box size=0.1 0.02 0.02
- added link WheelMarker_3, mass 0.01; visual box size=0.1 0.02 0.02
- added link WheelMarker_4, mass 0.01; visual box size=0.1 0.02 0.02
- added link WheelMarker_5, mass 0.01; visual box size=0.1 0.02 0.02
- added link WheelMarker_6, mass 0.01; visual box size=0.1 0.02 0.02
Joints:
- added joint $fixed_InertialWheel_1_WheelMarker_1: type fixed, parent InertialWheel_1, child WheelMarker_1, origin xyz=0 0 0.0001 rpy=0 0 0
- added joint $fixed_InertialWheel_2_WheelMarker_2: type fixed, parent InertialWheel_2, child WheelMarker_2, origin xyz=0 0 0.0001 rpy=0 0 0
- added joint $fixed_InertialWheel_3_WheelMarker_3: type fixed, parent InertialWheel_3, child WheelMarker_3, origin xyz=0 0 0.0001 rpy=0 0 0
- added joint $fixed_InertialWheel_4_WheelMarker_4: type fixed, parent InertialWheel_4, child WheelMarker_4, origin xyz=0 0 0.0001 rpy=0 0 0
- added joint $fixed_InertialWheel_5_WheelMarker_5: type fixed, parent InertialWheel_5, child WheelMarker_5, origin xyz=0 0 0.0001 rpy=0 0 0
- added joint $fixed_InertialWheel_6_WheelMarker_6: type fixed, parent InertialWheel_6, child WheelMarker_6, origin xyz=0 0 0.0001 rpy=0 0 0

File: assets/xacro/CubeBot.xacro (robot description, xacro)
@@ -112,4 +112,22 @@
         </link>
     </xacro:macro>
+    <xacro:macro name="WheelMarker" params="id_num cname color">
+        <link name="WheelMarker_${id_num}">
+            <visual>
+                <origin xyz="0 0 0" rpy="0 0 0"/>
+                <geometry>
+                    <box size="${WheelRadius2*1.25} ${WheelHeight*2} ${WheelHeight*2}"/>
+                </geometry>
+                <!-- <contact_coefficient mu="0"  resitution="0"  k_p="0"  k_d="0" /> -->
+                <material name="${cname}">
+                    <color rgba="${color}"/>
+                </material>
+            </visual>
+            <inertial>
+                <origin xyz="0 0 0" rpy="0 0 0"/>
+                <mass value="0.01"/>
+            </inertial>
+        </link>
+    </xacro:macro>
     <!-- Joint Definitions -->
     <xacro:macro name="fixedJoint" params="parent child pos rot">
@@ -145,4 +163,10 @@
     <xacro:InertialWheel id_num = "5" cname="Orange" color="${Orange}" />
     <xacro:InertialWheel id_num = "6" cname="Orange" color="${Orange}" />
+    <xacro:WheelMarker id_num = "1" cname="Blue" color="${Blue}" />
+    <xacro:WheelMarker id_num = "2" cname="Blue" color="${Blue}" />
+    <xacro:WheelMarker id_num = "3" cname="Blue" color="${Blue}" />
+    <xacro:WheelMarker id_num = "4" cname="Blue" color="${Blue}" />
+    <xacro:WheelMarker id_num = "5" cname="Blue" color="${Blue}" />
+    <xacro:WheelMarker id_num = "6" cname="Blue" color="${Blue}" />
     <!-- Joints -->
     <xacro:fixedJoint parent="CubeBody" child="CornerBumper_1" pos="${CornerOffset} ${CornerOffset} ${CornerOffset}" rot="0 0 0" />
@@ -160,3 +184,9 @@
     <xacro:continuous parent="CubeBody" child="InertialWheel_5" pos="0 0 ${WheelOffset}" rot="0 0 1.57075"  axis="0 0 1" damp="0" fric="0" />
     <xacro:continuous parent="CubeBody" child="InertialWheel_6" pos="0 0 -${WheelOffset}" rot="0 0 1.57075"  axis="0 0 1" damp="0" fric="0" />
+    <xacro:fixedJoint parent="InertialWheel_1" child="WheelMarker_1" pos="0 0 0.0001" rot="0 0 0" />
+    <xacro:fixedJoint parent="InertialWheel_2" child="WheelMarker_2" pos="0 0 0.0001" rot="0 0 0" />
+    <xacro:fixedJoint parent="InertialWheel_3" child="WheelMarker_3" pos="0 0 0.0001" rot="0 0 0" />
+    <xacro:fixedJoint parent="InertialWheel_4" child="WheelMarker_4" pos="0 0 0.0001" rot="0 0 0" />
+    <xacro:fixedJoint parent="InertialWheel_5" child="WheelMarker_5" pos="0 0 0.0001" rot="0 0 0" />
+    <xacro:fixedJoint parent="InertialWheel_6" child="WheelMarker_6" pos="0 0 0.0001" rot="0 0 0" />
 </robot>
